File: iotrain/iotrain.kicad_sch (KiCad schematic)
At the start: 68 parts, among them J1 12V, J10 X2, J11 SCL, J12 SDA, J13 GND, J14 3V3, J15 GND, J16 USB_B_Micro, J2 PROG ESP, J3 AC1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

Commit message: Make it smaller
Parts:
- removed C13: 10u/20V, Capacitor_SMD:C_0402_1005Metric, symbol Device:C
- added R11, R12: 1k, liebler_PASSIVES:SMD0201, symbol Device:R
- C1, C10, C14, C16, C19, C2, C21, C25, C26, C3, C4, C5, C6, C7, C8, C9: footprint Capacitor_SMD:C_0201_0603Metric -> liebler_PASSIVES:SMD0201
- C11: footprint Capacitor_SMD:C_0402_1005Metric -> Capacitor_SMD:C_0805_2012Metric
- C12, C18: footprint Capacitor_SMD:C_0201_0603Metric -> liebler_PASSIVES:SMD0402
- C15, C17, C20, C22: footprint Capacitor_SMD:C_0402_1005Metric -> liebler_PASSIVES:SMD0402
- L1, L2: footprint Inductor_SMD:L_0201_0603Metric -> liebler_PASSIVES:SMD0201
- R1, R10, R2, R3, R4, R5, R6, R7, R8, R9: footprint Resistor_SMD:R_0201_0603Metric -> liebler_PASSIVES:SMD0201
- SW1, SW2: footprint Button_Switch_SMD:SW_SPST_B3U-1000P -> liebler_MECH:SW_SPST_TL3342_smaller_handsolder
Connections:
- net PROG_EN is gone; now on net CHIP_EN: C21.1, R7.2, R8.1
- net +3V3: now also R11.2, R12.2
- net GND: now also R5.1
- net SCL: now also R11.1
- net SDA: now also R12.1

Commit message: Beautified
Parts:
- AE1: value Antenna_Chip -> Antenna
Connections:
- net +3V3: now also R8.1, U6.7 (VCC), U6.8 (LEDA); no longer R8.2
- net CHIP_EN: now also R8.2; no longer R8.1
- net GND: now also U6.10 (GND), U6.6 (GND)
- net LCD_BL: now also U6.9 (LEDK)
- net LCD_C: now also U6.2 (SCL)
- net LCD_CS: now also U6.5 (CS)
- net LCD_D: now also U6.1 (SDA)
- net LCD_RES: now also U6.4 (RES)
- net LCD_RS: now also U6.3 (RS)
Other:
- note added: "Audio"
- note added: "CPU"
- note added: "Connectors"
- note added: "Display"
- note added: "I2C"
- note added: "Motor Driver"
- note added: "PSU"
- note added: "Power MosFet"
- note added: "Rectifier"
- note added: "Switches"
- moved on the sheet: AE1, C1, C11, C15, C16, C17, C18, C19, C2, C20, C21, C22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

Commit message: various
Parts:
- added C13, C23: u1, liebler_PASSIVES:SMD0201, symbol Device:C
- added D6, D7: XL-1010RGBC-WS2812B, liebler_OPTO:XL-1010RGBC-WS2812B, symbol liebler_OPTO:XL-1010RGBC-WS2812B
- C11: value 10u/20V -> 22u/25V; footprint Capacitor_SMD:C_0805_2012Metric -> liebler_PASSIVES:SMD0805
- C15, C20, C22: value 10u/20V -> 10u/25V; footprint liebler_PASSIVES:SMD0402 -> liebler_PASSIVES:SMD0603
- SW1, SW2: footprint liebler_MECH:SW_SPST_TL3342_smaller_handsolder -> Button_Switch_SMD:SW_Push_SPST_NO_Alps_SKRK
Connections:
- net +3V3: now also C13.2, C23.2, D6.2 (VDD), D7.2 (VDD)
- net GND: now also C13.1, C23.1, D6.3 (VSS), D7.3 (VSS)
- net RGB_LED: now reaches U4.25 (GPIO20/SDIO_DATA0/FSPICS4)
- net RGB_LED: now also D6.4 (DIN)
- new net: D6.1 (DOUT), D7.4 (DIN)
